Commit message: RP-248 Fix materials

File: urdf/materials.urdf.xacro (robot description, xacro)
@@ -35,8 +35,8 @@
 		<color rgba="0.0 0.8 0.0 1.0"/>
 	</material>
-	<material name="Gray">
+	<material name="Grey">
 		<color rgba="0.7 0.7 0.7 1.0"/>
 	</material>
-	<material name="DarkGray">
+	<material name="DarkGrey">
 		<color rgba="0.3 0.3 0.3 1.0"/>
 	</material>

File: urdf/parts.urdf.xacro (robot description, xacro)
@@ -55,5 +55,5 @@
         <mesh filename="package://husky_description/meshes/user_rail.stl" />
       </geometry>
-      <material name="DarkGray" />
+      <material name="DarkGrey" />
     </visual>
   </link>
@@ -64,5 +64,5 @@
   </joint>
   <gazebo reference="user_rail_link">
-    <material>Gazebo/DarkGray</material>
+    <material>Gazebo/DarkGrey</material>
   </gazebo>
   <link name="front_bumper_link">
@@ -71,5 +71,5 @@
         <mesh filename="package://husky_description/meshes/bumper.stl" />
       </geometry>
-      <material name="DarkGray" />
+      <material name="DarkGrey" />
     </visual>
   </link>
@@ -80,5 +80,5 @@
   </joint>
   <gazebo reference="front_bumper_link">
-    <material>Gazebo/DarkGray</material>
+    <material>Gazebo/DarkGrey</material>
   </gazebo>
   <link name="rear_bumper_link">
@@ -87,5 +87,5 @@
         <mesh filename="package://husky_description/meshes/bumper.stl" />
       </geometry>
-      <material name="DarkGray" />
+      <material name="DarkGrey" />
     </visual>
   </link>
@@ -96,5 +96,5 @@
   </joint>
   <gazebo reference="rear_bumper_link">
-    <material>Gazebo/DarkGray</material>
+    <material>Gazebo/DarkGrey</material>
   </gazebo>
   <gazebo>
@@ -142,5 +142,5 @@
           <mesh filename="package://husky_description/meshes/lidar_mount.stl" />
         </geometry>
-        <material name="DarkGray" />
+        <material name="DarkGrey" />
       </visual>
     </link>
@@ -151,5 +151,5 @@
     </joint>
     <gazebo reference="sick_bracket_link">
-      <material>Gazebo/DarkGray</material>
+      <material>Gazebo/DarkGrey</material>
     </gazebo>
     <xacro:sick_lms100 prefix="front" />

File: urdf/sensors/sick_lms100.urdf.xacro (robot description, xacro)
@@ -50,5 +50,5 @@
           <mesh filename="package://husky_description/meshes/sick_lms100.stl" />
         </geometry>
-        <material name="light_grey" />
+        <material name="Grey" />
       </visual>
       <collision>

File: urdf/wheel.urdf.xacro (robot description, xacro)
@@ -39,10 +39,10 @@
 					<mesh filename="package://husky_description/meshes/wheel.stl" />
 				</geometry>
-				<material name="DarkGray" />
+				<material name="DarkGrey" />
 			</visual>
 			<collision>
 				<origin xyz="0 0 0" rpy="${M_PI/2} 0 0" />
 				<geometry>
-				    <cylinder length="0.1143" radius="0.3555" />
+				    <cylinder length="0.1143" radius="0.17775" />
 				</geometry>
 			</collision>
