Commit message: RP-248 fix standard angle for imu

File: urdf/parts.urdf.xacro (robot description, xacro)
@@ -36,5 +36,5 @@
   <link name="imu_link"/>
   <joint name="imu_joint" type="fixed">
-    <origin xyz="$(optenv HUSKY_IMU_XYZ 0.25 0 0.0415)" rpy="$(optenv HUSKY_IMU_RPY 0 -1.57 0)" />
+    <origin xyz="$(optenv HUSKY_IMU_XYZ 0.25 0 0.0415)" rpy="$(optenv HUSKY_IMU_RPY 3.141 -1.5705 0)" />
     <parent link="chassis_link" />
     <child link="imu_link" />

Commit message: RP-248 Restore default imu transform

File: urdf/parts.urdf.xacro (robot description, xacro)
@@ -36,5 +36,5 @@
   <link name="imu_link"/>
   <joint name="imu_joint" type="fixed">
-    <origin xyz="$(optenv HUSKY_IMU_XYZ 0.25 0 0.0415)" rpy="$(optenv HUSKY_IMU_RPY 3.141 -1.5705 0)" />
+    <origin xyz="$(optenv HUSKY_IMU_XYZ 0.25 0 0.0415)" rpy="$(optenv HUSKY_IMU_RPY 0 1.5708 1.5708)" />
     <parent link="chassis_link" />
     <child link="imu_link" />
