Commit message: combining xacro files to include sensors in the default xacro with enable flags

File: urdf/base.urdf.xacro (robot description, xacro)
@@ -18,4 +18,6 @@
     <xacro:include filename="$(find husky_description)/urdf/wheel.urdf.xacro" />
     <xacro:include filename="$(find husky_description)/urdf/parts.urdf.xacro" />
+    <xacro:include filename="$(find husky_description)/urdf/sensors/sick_laser.urdf.xacro" />
+    <xacro:include filename="$(find husky_description)/urdf/sensors/gps.urdf.xacro" />
 	<!-- PROPERTY LIST -->
     <!--All units in m-kg-s-radians unit system -->
@@ -142,4 +144,44 @@
             <torque>35</torque>
         </plugin>
+      </gazebo>
+  <xacro:if value="$(arg imu_enabled)">
+    <gazebo>
+      <plugin name="imu_plugin" filename="libgazebo_ros_imu.so">
+        <alwaysOn>true</alwaysOn>
+        <bodyName>base_link</bodyName>
+        <topicName>imu_data</topicName>
+        <serviceName>imu_service</serviceName>
+        <gaussianNoise>0.01</gaussianNoise>
+      </plugin>
     </gazebo>
+  </xacro:if>
+  <xacro:if value="$(arg gps_enabled)">
+    <gazebo>
+      <plugin name="gps_plugin" filename="libhusky_tudarmstadt_gps_plugin.so">
+      <alwaysOn>true</alwaysOn>
+          <updateRate>4.0</updateRate>
+          <bodyName>base_link</bodyName>
+          <topicName>navsat/fix</topicName>
+          <velocityTopicName>navsat/fix_velocity</velocityTopicName>
+          <drift>0.1 0.1 0.1</drift>
+          <gaussianNoise>0.01 0.01 0.01</gaussianNoise>
+          <velocityDrift>0 0 0</velocityDrift>
+          <velocityGaussianNoise>0.1 0.1 0.1</velocityGaussianNoise>
+          <referenceLatitude>43.409991</referenceLatitude>
+          <referenceLongitude>-80.448362</referenceLongitude>
+      </plugin>
+  </gazebo>
+  </xacro:if>
+  <xacro:if value="$(arg lidar_enabled)">
+    <husky_part parent="base_footprint" name="user_plate" mesh="user_plate"
+      colour="DarkGray"
+      translateX="-0.35" translateY="-0.325" translateZ="${0.165 + wheel_x_size/2 - base_z_origin_to_wheel_origin}"
+      rotateX="1.5705" rotateY="0.0" rotateZ="1.5705"/>
+    <gazebo reference="base_footprint_user_plate_part">
+      <material>Gazebo/FlatBlack</material>
+    </gazebo>
+    <!-- This adds the laser macro, including the scan for gazebo and link name -->
+  <sick_laser_v0 name="laser" parent="base" ros_topic="scan"
+    update_rate="20" min_angle="-1.57" max_angle="1.57" />
+  </xacro:if>
 </robot>

Commit message: cleanup and parameterization of files and lidar mounting

File: urdf/base.urdf.xacro (robot description, xacro)
@@ -1,18 +1,6 @@
 <?xml version="1.0"?>
 <robot
-	xmlns:xi="http://www.w3.org/2001/XInclude"
-	xmlns:gazebo="http://playerstage.sourceforge.net/gazebo/xmlschema/#gz"
-    xmlns:model="http://playerstage.sourceforge.net/gazebo/xmlschema/#model"
-	xmlns:sensor="http://playerstage.sourceforge.net/gazebo/xmlschema/#sensor"
-	xmlns:body="http://playerstage.sourceforge.net/gazebo/xmlschema/#body"
-    xmlns:geom="http://playerstage.sourceforge.net/gazebo/xmlschema/#geom"
-    xmlns:joint="http://playerstage.sourceforge.net/gazebo/xmlschema/#joint"
-	xmlns:controller="http://playerstage.sourceforge.net/gazebo/xmlschema/#controller"
-	xmlns:interface="http://playerstage.sourceforge.net/gazebo/xmlschema/#interface"
-	xmlns:rendering="http://playerstage.sourceforge.net/gazebo/xmlschema/#rendering"
-    xmlns:renderable="http://playerstage.sourceforge.net/gazebo/xmlschema/#renderable"
-    xmlns:physics="http://playerstage.sourceforge.net/gazebo/xmlschema/#physics"
-	xmlns:xacro="http://ros.org/wiki/xacro" name="husky">
-	<!-- Included URDF/XACRO Files -->
+	xmlns:xi="http://www.w3.org/2001/XInclude" xmlns:xacro="http://ros.org/wiki/xacro" name="husky">
+    <!-- Included URDF/XACRO Files -->
     <xacro:include filename="$(find husky_description)/urdf/materials.urdf.xacro" />
     <xacro:include filename="$(find husky_description)/urdf/wheel.urdf.xacro" />
@@ -20,5 +8,5 @@
     <xacro:include filename="$(find husky_description)/urdf/sensors/sick_laser.urdf.xacro" />
     <xacro:include filename="$(find husky_description)/urdf/sensors/gps.urdf.xacro" />
-	<!-- PROPERTY LIST -->
+  	<!-- PROPERTY LIST -->
     <!--All units in m-kg-s-radians unit system -->
     <property name="M_PI" value="3.1415926535897931" />
@@ -41,5 +29,5 @@
     <property name="base_iyz_com_cs" value="-0.00154437" />
     <property name="base_izz_com_cs" value="2.02955229" />
-<!-- BASE-FOOTPRINT -->
+    <!-- BASE-FOOTPRINT -->
     <!-- base_footprint is a fictitious link(frame) that is on the ground right below base_link origin, navigation stack depends on this frame -->
     <link name="base_footprint">
@@ -183,5 +171,8 @@
     <!-- This adds the laser macro, including the scan for gazebo and link name -->
   <sick_laser_v0 name="laser" parent="base" ros_topic="scan"
-    update_rate="20" min_angle="-1.57" max_angle="1.57" />
+    update_rate="20" min_angle="-1.57" max_angle="1.57" l_x="0.5" l_y="0.0" l_z="0.25" l_r="0.0" l_p="0.0" l_yaw="0.0"/>
+    <gazebo reference="laser_link">
+      <material>Gazebo/FlatBlack</material>
+    </gazebo>
   </xacro:if>
 </robot>

File: urdf/sensors/gps.urdf.xacro (robot description, xacro)
@@ -1,10 +1,5 @@
 <?xml version="1.0"?>
-<robot xmlns:sensor="http://playerstage.sourceforge.net/gazebo/xmlschema/#sensor"
-       xmlns:controller="http://playerstage.sourceforge.net/gazebo/xmlschema/#controller"
-       xmlns:interface="http://playerstage.sourceforge.net/gazebo/xmlschema/#interface"
-      xmlns:plugin="http://playerstage.sourceforge.net/gazebo/xmlschema/#plugin"
-       xmlns:xacro="http://ros.org/wiki/xacro">
+<robot xmlns:xacro="http://ros.org/wiki/xacro">
   <xacro:macro name="novatel_gps_sensor" params="name gps_topic velocity_topic lat lon">
-  <!-- This adds a visual box to allow us to see the GPS in rviz/gazebo -->
     <joint name="gps_joint" type="fixed">
       <origin xyz="0.39 0.385 0.10" rpy="-1.5705 -1.5705 0" />
@@ -13,23 +8,17 @@
     </joint>
     <link name="gps_link">
-      <inertial>
-        <mass value="0.01" />
-        <origin xyz="0 0 0" />
-        <inertia ixx="0.001"  ixy="0.0"  ixz="0.0"
-        iyy="0.001"  iyz="0.0"
-        izz="0.001" />
-      </inertial>
-      <visual>
-        <origin xyz="0 0 0.1" rpy="1.5705 0 -1.5705"/>
-        <geometry>
-        <mesh filename="package://husky_description/meshes/gps.stl" />
-        </geometry>
-      </visual>
-      <collision>
-        <origin xyz="0 0 0" rpy="0 0 0"/>
-        <geometry>
-        <mesh filename="package://husky_description/meshes/gps.stl" />
-        </geometry>
-      </collision>
+    <inertial>
+      <mass value="0.01" />
+      <origin xyz="0 0 0" />
+      <inertia ixx="0.001"  ixy="0.0"  ixz="0.0"
+      iyy="0.001"  iyz="0.0"
+      izz="0.001" />
+    </inertial>
+    <visual>
+      <origin xyz="0 0 0.1" rpy="1.5705 0 -1.5705"/>
+    </visual>
+    <collision>
+      <origin xyz="0 0 0" rpy="0 0 0"/>
+    </collision>
     </link>
   </xacro:macro>

File: urdf/sensors/sick_laser.urdf.xacro (robot description, xacro)
@@ -1,38 +1,35 @@
 <?xml version="1.0"?>
-<robot xmlns:sensor="http://playerstage.sourceforge.net/gazebo/xmlschema/#sensor"
-       xmlns:controller="http://playerstage.sourceforge.net/gazebo/xmlschema/#controller"
-       xmlns:interface="http://playerstage.sourceforge.net/gazebo/xmlschema/#interface"
-       xmlns:xacro="http://ros.org/wiki/xacro">
-       <xacro:include filename="$(find husky_description)/urdf/sensors/sick_laser.gazebo.xacro" />
-  <xacro:macro name="sick_laser_v0" params="name parent ros_topic update_rate min_angle max_angle">
-        <!-- This adds a visual box to allow us to see the Hokuyo in rviz/gazebo -->
-        <joint name="laser_scan_joint" type="fixed">
-          <origin xyz="0.3 0 0.4" rpy="0 0 0" />
-          <parent link="base_link" />
-          <child link="${name}_link"/>
-        </joint>
-       <link name="${name}_link">
-          <inertial>
-            <mass value="0.01" />
-            <origin xyz="0 0 0" />
-            <inertia ixx="0.001"  ixy="0.0"  ixz="0.0"
-            iyy="0.001"  iyz="0.0"
-                izz="0.001" />
-          </inertial>
-            <visual>
-                <origin xyz="0 0 0.1" rpy="1.5705 0 -1.5705"/>
-                <geometry>
-                    <mesh filename="package://husky_description/meshes/lidar.stl" />
-                </geometry>
-            </visual>
-            <collision>
-                <origin xyz="0 0 0" rpy="0 0 0"/>
-                <geometry>
-                  <mesh filename="package://husky_description/meshes/lidar.stl" />
-                </geometry>
-            </collision>
-        </link>
+  <robot xmlns:xacro="http://ros.org/wiki/xacro">
+  <xacro:include filename="$(find husky_description)/urdf/sensors/sick_laser.gazebo.xacro" />
+  <xacro:macro name="sick_laser_v0" params="name parent ros_topic update_rate min_angle max_angle l_x l_y l_z l_r l_p l_yaw">
+    <!-- This adds a visual box to allow us to see the Hokuyo in rviz/gazebo -->
+    <joint name="laser_scan_joint" type="fixed">
+      <origin xyz="${l_x} ${l_y} ${l_z}" rpy="${l_r} ${l_p} ${l_yaw}" />
+      <parent link="${parent}_link" />
+      <child link="${name}_link"/>
+    </joint>
+    <link name="${name}_link">
+      <inertial>
+        <mass value="0.01" />
+        <origin xyz="0 0 0" />
+        <inertia ixx="0.001"  ixy="0.0"  ixz="0.0"
+        iyy="0.001"  iyz="0.0"
+            izz="0.001" />
+      </inertial>
+      <visual>
+          <origin xyz="0 0 0.1" rpy="1.5705 0 -1.5705"/>
+          <geometry>
+              <mesh filename="package://husky_description/meshes/lidar.stl" />
+          </geometry>
+      </visual>
+      <collision>
+          <origin xyz="0 0 0" rpy="0 0 0"/>
+          <geometry>
+            <mesh filename="package://husky_description/meshes/lidar.stl" />
+          </geometry>
+      </collision>
+    </link>
     <!-- gazebo extensions -->
     <xacro:sick_laser_gazebo_v0 name="${name}" ros_topic="${ros_topic}" update_rate="${update_rate}" min_angle="${min_angle}" max_angle="${max_angle}" />
-  </xacro:macro>
+    </xacro:macro>
 </robot>

Commit message: fixing how the lidar is mounted to make sure its consistent with the collision model and that the LIDAR rays don't hit the body itself

File: urdf/base.urdf.xacro (robot description, xacro)
@@ -75,5 +75,5 @@
 			<origin xyz="0 0 ${wheel_x_size/2 - base_z_origin_to_wheel_origin - 0.02}" rpy="0 0 0 " />
 			<geometry>
-				<box size = "${base_x_size+0.02} ${base_y_size} ${base_z_size + 0.02}"/> <!--making it slightly bigger in x and z direction-->
+        <box size = "${base_x_size+0.02} ${base_y_size} ${base_z_size + 0.02}"/> <!--making it slightly bigger in x and z direction-->
 			</geometry>
 		</collision>
@@ -171,5 +171,5 @@
     <!-- This adds the laser macro, including the scan for gazebo and link name -->
   <sick_laser_v0 name="laser" parent="base" ros_topic="scan"
-    update_rate="20" min_angle="-1.57" max_angle="1.57" l_x="0.5" l_y="0.0" l_z="0.25" l_r="0.0" l_p="0.0" l_yaw="0.0"/>
+    update_rate="20" min_angle="-1.57" max_angle="1.57" l_x="0.5" l_y="0.0" l_z="0.3" l_r="0.0" l_p="0.0" l_yaw="0.0"/>
     <gazebo reference="laser_link">
       <material>Gazebo/FlatBlack</material>

File: urdf/sensors/sick_laser.urdf.xacro (robot description, xacro)
@@ -12,5 +12,5 @@
       <inertial>
         <mass value="0.01" />
-        <origin xyz="0 0 0" />
+        <origin xyz="0 0 0.3" />
         <inertia ixx="0.001"  ixy="0.0"  ixz="0.0"
         iyy="0.001"  iyz="0.0"
@@ -18,5 +18,5 @@
       </inertial>
       <visual>
-          <origin xyz="0 0 0.1" rpy="1.5705 0 -1.5705"/>
+          <origin xyz="0 0 0" rpy="1.5705 0 -1.5705"/>
           <geometry>
               <mesh filename="package://husky_description/meshes/lidar.stl" />
@@ -24,5 +24,5 @@
       </visual>
       <collision>
-          <origin xyz="0 0 0" rpy="0 0 0"/>
+          <origin xyz="0 0 0" rpy="1.5705 0 -1.5705"/>
           <geometry>
             <mesh filename="package://husky_description/meshes/lidar.stl" />

Commit message: removing ugly user_plate, adding proper lidar mount instead

File: urdf/base.urdf.xacro (robot description, xacro)
@@ -83,9 +83,9 @@
         <turnGravityOff>false</turnGravityOff>
     </gazebo>
-    <!-- WHEEL macros -->
-	<husky_wheel fb="back" lr="left" parent="base_link" translateX="-1" translateY="1" flipY="-1"/>
-	<husky_wheel fb="back" lr="right" parent="base_link" translateX="-1" translateY="-1" flipY="-1"/>
-	<husky_wheel fb="front" lr="left" parent="base_link" translateX="1" translateY="1" flipY="-1"/>
-	<husky_wheel fb="front" lr="right" parent="base_link" translateX="1" translateY="-1" flipY="-1"/>
+      <!-- WHEEL macros -->
+    <husky_wheel fb="back" lr="left" parent="base_link" translateX="-1" translateY="1" flipY="-1"/>
+    <husky_wheel fb="back" lr="right" parent="base_link" translateX="-1" translateY="-1" flipY="-1"/>
+    <husky_wheel fb="front" lr="left" parent="base_link" translateX="1" translateY="1" flipY="-1"/>
+    <husky_wheel fb="front" lr="right" parent="base_link" translateX="1" translateY="-1" flipY="-1"/>
     <!-- DECORATIONS -->
     <!-- Top Plate -->
@@ -106,11 +106,11 @@
     </gazebo>
     <!-- Bumpers -->
-    <husky_part parent="base_footprint" name="front_bumper" mesh="bumper"
+    <husky_part parent="base_footprint" name="front_bumper" mesh="front_bumper"
           colour="DarkGray"
-          translateX="0.490" translateY="0.0" translateZ="${0.091 + wheel_x_size/2 - base_z_origin_to_wheel_origin}"
+          translateX="0.530" translateY="0.0" translateZ="${0.091 + wheel_x_size/2 - base_z_origin_to_wheel_origin}"
           rotateX="0.0" rotateY="0.0" rotateZ="0.0"/>
     <gazebo reference="base_footprint_front_bumper_part">
         <material>Gazebo/FlatBlack</material>
-    </gazebo>
+      </gazebo>
     <husky_part parent="base_footprint" name="rear_bumper" mesh="bumper"
           colour="DarkGray"
@@ -162,17 +162,17 @@
   </xacro:if>
   <xacro:if value="$(arg lidar_enabled)">
-    <husky_part parent="base_footprint" name="user_plate" mesh="user_plate"
+    <husky_part parent="base_footprint_front_bumper_part" name="sick_bracket" mesh="lidar_mount"
       colour="DarkGray"
-      translateX="-0.35" translateY="-0.325" translateZ="${0.165 + wheel_x_size/2 - base_z_origin_to_wheel_origin}"
-      rotateX="1.5705" rotateY="0.0" rotateZ="1.5705"/>
-    <gazebo reference="base_footprint_user_plate_part">
+      translateX="-0.12" translateY="0" translateZ="0"
+      rotateX="0" rotateY="0.0" rotateZ="0"/>
+    <gazebo reference="lidar_mount_bracket_part">
       <material>Gazebo/FlatBlack</material>
     </gazebo>
     <!-- This adds the laser macro, including the scan for gazebo and link name -->
-  <sick_laser_v0 name="laser" parent="base" ros_topic="scan"
-    update_rate="20" min_angle="-1.57" max_angle="1.57" l_x="0.5" l_y="0.0" l_z="0.3" l_r="0.0" l_p="0.0" l_yaw="0.0"/>
-    <gazebo reference="laser_link">
-      <material>Gazebo/FlatBlack</material>
-    </gazebo>
+    <sick_laser_v0 name="laser" parent="base_footprint_front_bumper_part_sick_bracket_part" ros_topic="scan"
+      update_rate="20" min_angle="-1.57" max_angle="1.57" l_x="0.055" l_y="0.0" l_z="0.17" l_r="${M_PI}" l_p="0.0" l_yaw="0.0"/>
+      <gazebo reference="laser_link">
+        <material>Gazebo/White</material>
+      </gazebo>
   </xacro:if>
 </robot>

File: urdf/sensors/sick_laser.urdf.xacro (robot description, xacro)
@@ -6,5 +6,5 @@
     <joint name="laser_scan_joint" type="fixed">
       <origin xyz="${l_x} ${l_y} ${l_z}" rpy="${l_r} ${l_p} ${l_yaw}" />
-      <parent link="${parent}_link" />
+      <parent link="${parent}" />
       <child link="${name}_link"/>
     </joint>
@@ -18,5 +18,5 @@
       </inertial>
       <visual>
-          <origin xyz="0 0 0" rpy="1.5705 0 -1.5705"/>
+          <origin xyz="0 0 0.03" rpy="1.5705 0 -1.5705"/>
           <geometry>
               <mesh filename="package://husky_description/meshes/lidar.stl" />
@@ -24,5 +24,5 @@
       </visual>
       <collision>
-          <origin xyz="0 0 0" rpy="1.5705 0 -1.5705"/>
+          <origin xyz="0 0 0.03" rpy="1.5705 0 -1.5705"/>
           <geometry>
             <mesh filename="package://husky_description/meshes/lidar.stl" />

Commit message: cleanup of some lidar files, by leveraging new jackal work. now the LIDAR transforms are consistent

File: urdf/base.urdf.xacro (robot description, xacro)
@@ -6,6 +6,6 @@
     <xacro:include filename="$(find husky_description)/urdf/wheel.urdf.xacro" />
     <xacro:include filename="$(find husky_description)/urdf/parts.urdf.xacro" />
-    <xacro:include filename="$(find husky_description)/urdf/sensors/sick_laser.urdf.xacro" />
     <xacro:include filename="$(find husky_description)/urdf/sensors/gps.urdf.xacro" />
+  <xacro:include filename="sensors/sick_lms100.urdf.xacro" />
   	<!-- PROPERTY LIST -->
     <!--All units in m-kg-s-radians unit system -->
@@ -133,33 +133,33 @@
         </plugin>
       </gazebo>
-  <xacro:if value="$(arg imu_enabled)">
-    <gazebo>
-      <plugin name="imu_plugin" filename="libgazebo_ros_imu.so">
-        <alwaysOn>true</alwaysOn>
-        <bodyName>base_link</bodyName>
-        <topicName>imu_data</topicName>
-        <serviceName>imu_service</serviceName>
-        <gaussianNoise>0.01</gaussianNoise>
-      </plugin>
-    </gazebo>
-  </xacro:if>
-  <xacro:if value="$(arg gps_enabled)">
-    <gazebo>
-      <plugin name="gps_plugin" filename="libhusky_tudarmstadt_gps_plugin.so">
-      <alwaysOn>true</alwaysOn>
-          <updateRate>4.0</updateRate>
-          <bodyName>base_link</bodyName>
-          <topicName>navsat/fix</topicName>
-          <velocityTopicName>navsat/fix_velocity</velocityTopicName>
-          <drift>0.1 0.1 0.1</drift>
-          <gaussianNoise>0.01 0.01 0.01</gaussianNoise>
-          <velocityDrift>0 0 0</velocityDrift>
-          <velocityGaussianNoise>0.1 0.1 0.1</velocityGaussianNoise>
-          <referenceLatitude>43.409991</referenceLatitude>
-          <referenceLongitude>-80.448362</referenceLongitude>
-      </plugin>
-  </gazebo>
-  </xacro:if>
-  <xacro:if value="$(arg lidar_enabled)">
+	  <xacro:if value="$(arg imu_enabled)">
+	    <gazebo>
+	      <plugin name="imu_plugin" filename="libgazebo_ros_imu.so">
+		<alwaysOn>true</alwaysOn>
+		<bodyName>base_link</bodyName>
+		<topicName>imu_data</topicName>
+		<serviceName>imu_service</serviceName>
+		<gaussianNoise>0.01</gaussianNoise>
+	      </plugin>
+	    </gazebo>
+	  </xacro:if>
+	  <xacro:if value="$(arg gps_enabled)">
+	    <gazebo>
+	      <plugin name="gps_plugin" filename="libhusky_tudarmstadt_gps_plugin.so">
+	      <alwaysOn>true</alwaysOn>
+		  <updateRate>4.0</updateRate>
+		  <bodyName>base_link</bodyName>
+		  <topicName>navsat/fix</topicName>
+		  <velocityTopicName>navsat/fix_velocity</velocityTopicName>
+		  <drift>0.1 0.1 0.1</drift>
+		  <gaussianNoise>0.01 0.01 0.01</gaussianNoise>
+		  <velocityDrift>0 0 0</velocityDrift>
+		  <velocityGaussianNoise>0.1 0.1 0.1</velocityGaussianNoise>
+		  <referenceLatitude>43.409991</referenceLatitude>
+		  <referenceLongitude>-80.448362</referenceLongitude>
+	      </plugin>
+	  </gazebo>
+	  </xacro:if>
+  <xacro:if value="$(arg front_laser)">
     <husky_part parent="base_footprint_front_bumper_part" name="sick_bracket" mesh="lidar_mount"
       colour="DarkGray"
@@ -169,10 +169,10 @@
       <material>Gazebo/FlatBlack</material>
     </gazebo>
-    <!-- This adds the laser macro, including the scan for gazebo and link name -->
-    <sick_laser_v0 name="laser" parent="base_footprint_front_bumper_part_sick_bracket_part" ros_topic="scan"
-      update_rate="20" min_angle="-1.57" max_angle="1.57" l_x="0.055" l_y="0.0" l_z="0.17" l_r="${M_PI}" l_p="0.0" l_yaw="0.0"/>
-      <gazebo reference="laser_link">
-        <material>Gazebo/White</material>
-      </gazebo>
-  </xacro:if>
+    <xacro:sick_lms100 prefix="front" />
+    <joint name="front_laser_joint" type="fixed">
+      <origin xyz="0.07 0 0.17" rpy="0 0 0" />
+      <parent link="base_footprint_front_bumper_part_sick_bracket_part" />
+      <child link="front_laser" />
+    </joint>
+ </xacro:if>
 </robot>
