Commit message: RP-248 Refactor description

File: urdf/base.urdf.xacro (robot description, xacro)
@@ -8,22 +8,13 @@
   <xacro:include filename="$(find husky_description)/urdf/sensors/sick_lms100.urdf.xacro" />
   <!-- PROPERTY LIST -->
-  <!-- <property name="M_PI" value="3.1415926535897931" /> -->
-  <!-- Location of center of mass. -->
-  <property name="base_x_com" value="-0.08748000" />
-  <property name="base_y_com" value="-0.00085000" />
-  <property name="base_z_com" value="0.09947000" />
+  <property name="M_PI" value="3.1415926535897931" />
   <!-- Size of the base. -->
   <property name="base_x_size" value="0.98740000" />
   <property name="base_y_size" value="0.57090000" />
   <property name="base_z_size" value="0.24750000" />
-  <!-- Weight of the base, kg. -->
-  <property name="base_mass" value="33.45489000" />
   <!-- Inertial values for the base at center of mass, aligned with coordinate system. Units are kg*m^2 -->
-  <property name="base_ixx_com_cs" value="0.60216370" />
-  <property name="base_ixy_com_cs" value="-0.02364198" />
-  <property name="base_ixz_com_cs" value="-0.11972132" />
-  <property name="base_iyy_com_cs" value="1.73859574" />
-  <property name="base_iyz_com_cs" value="-0.00154437" />
-  <property name="base_izz_com_cs" value="2.02955229" />
+  <xacro:property name="wheelbase" value="0.5120" />
+  <xacro:property name="track" value="0.5708" />
+  <xacro:property name="wheel_vertical_offset" value="0.03282" />
   <!-- Root node is the body of the robot. -->
   <link name="base_link">
@@ -36,5 +27,5 @@
     </visual>
     <collision>
-      <origin xyz="0 0 ${wheel_x_size/2 - base_z_origin_to_wheel_origin - 0.02}" rpy="0 0 0" />
+      <origin xyz="0 0 ${0.1578 - wheel_vertical_offset}" rpy="0 0 0" />
       <geometry>
         <!-- Make collision box slightly bigger in x and z directions. -->
@@ -43,12 +34,14 @@
     </collision>
   </link>
-  <!-- KDL can't have inertia on the base_link, so move it to this separate link. -->
+  <gazebo reference="base_link">
+    <material>Gazebo/DarkGrey</material>
+    <turnGravityOff>false</turnGravityOff>
+  </gazebo>
   <link name="base_inertia">
     <inertial>
-      <mass value="${base_mass}" />
-      <!-- This is the pose of the inertial reference frame, relative to the link reference frame. The origin of the inertial reference frame needs to be at the center of gravity. The axes of the inertial reference frame do not need to be aligned with the principal axes of the inertia.-->
-      <origin xyz="${base_x_com} ${base_y_com} ${base_z_com}" />
-      <inertia ixx="${base_ixx_com_cs}" ixy="${base_ixy_com_cs}" ixz="${base_ixz_com_cs}"
-       iyy="${base_iyy_com_cs}" iyz="${base_iyz_com_cs}" izz="${base_izz_com_cs}" />
+      <mass value="33.455" />
+      <origin xyz="-0.08748 -0.00085 0.09947" />
+      <inertia ixx="0.6022" ixy="-0.02364" ixz="-0.1197"
+       iyy="1.7386" iyz="-0.001544" izz="2.0296" />
      </inertial>
    </link>
@@ -58,97 +51,18 @@
     <child link="base_inertia" />
   </joint>
-  <gazebo reference="base_link">
-    <material>Gazebo/DarkGrey</material>
+  <gazebo reference="base_inertia">
     <turnGravityOff>false</turnGravityOff>
   </gazebo>
-  <!-- WHEEL macros -->
-  <husky_wheel fb="back" lr="left" parent="base_link" translateX="-1" translateY="1" flipY="-1"/>
-  <husky_wheel fb="back" lr="right" parent="base_link" translateX="-1" translateY="-1" flipY="-1"/>
-  <husky_wheel fb="front" lr="left" parent="base_link" translateX="1" translateY="1" flipY="-1"/>
-  <husky_wheel fb="front" lr="right" parent="base_link" translateX="1" translateY="-1" flipY="-1"/>
-  <!-- DECORATIONS -->
-  <!-- Top Plate -->
-  <husky_part parent="base_link" name="top_plate" mesh="top_plate"
-    colour="Yellow"
-    translateX="0.0" translateY="0.0" translateZ="0.0"
-    rotateX="0.0" rotateY="0.0" rotateZ="0.0"/>
-  <gazebo reference="base_link_top_plate_part">
-    <material>Gazebo/Yellow</material>
-  </gazebo>
-  <!-- User Rail -->
-  <husky_part parent="base_link" name="user_rail" mesh="user_rail"
-    colour="DarkGray"
-    translateX="0.272" translateY="0.0" translateZ="0.245"
-    rotateX="0.0" rotateY="0.0" rotateZ="0.0"/>
-  <gazebo reference="base_link_user_rail_part">
-    <material>Gazebo/DarkGrey</material>
-  </gazebo>
-  <!-- Bumpers -->
-  <husky_part parent="base_link" name="front_bumper" mesh="bumper"
-    colour="DarkGray"
-    translateX="0.48" translateY="0.0" translateZ="0.091"
-    rotateX="0.0" rotateY="0.0" rotateZ="0.0"/>
-  <gazebo reference="base_link_front_bumper_part">
-    <material>Gazebo/DarkGrey</material>
-  </gazebo>
-  <husky_part parent="base_link" name="rear_bumper" mesh="bumper"
-    colour="DarkGray"
-    translateX="-0.48" translateY="0.0" translateZ="0.091"
-    rotateX="0.0" rotateY="0.0" rotateZ="3.14"/>
-  <gazebo reference="base_link_rear_bumper_part">
-    <material>Gazebo/DarkGrey</material>
-  </gazebo>
-  <gazebo>
-    <plugin name="gazebo_ros_control" filename="libgazebo_ros_control.so">
-      <robotNamespace>/</robotNamespace>
-    </plugin>
-  </gazebo>
-  <xacro:if value="$(arg imu_enabled)">
-    <gazebo>
-      <plugin name="imu_controller" filename="libhector_gazebo_ros_imu.so">
-        <robotNamespace>/</robotNamespace>
-        <updateRate>50.0</updateRate>
-        <bodyName>base_link</bodyName>
-        <topicName>imu/data</topicName>
-        <accelDrift>0.005 0.005 0.005</accelDrift>
-        <accelGaussianNoise>0.005 0.005 0.005</accelGaussianNoise>
-        <rateDrift>0.005 0.005 0.005 </rateDrift>
-        <rateGaussianNoise>0.005 0.005 0.005 </rateGaussianNoise>
-        <headingDrift>0.005</headingDrift>
-        <headingGaussianNoise>0.005</headingGaussianNoise>
-      </plugin>
-    </gazebo>
-  </xacro:if>
-  <xacro:if value="$(arg gps_enabled)">
-    <gazebo>
-      <plugin name="gps_controller" filename="libhector_gazebo_ros_gps.so">
-        <updateRate>40</updateRate>
-        <robotNamespace>/</robotNamespace>
-        <bodyName>base_link</bodyName>
-        <frameId>base_link</frameId>
-        <topicName>/navsat/fix</topicName>
-        <velocityTopicName>/navsat/vel</velocityTopicName>
-        <referenceLatitude>49.9</referenceLatitude>
-        <referenceLongitude>8.9</referenceLongitude>
-        <referenceHeading>0</referenceHeading>
-        <referenceAltitude>0</referenceAltitude>
-        <drift>0.0001 0.0001 0.0001</drift>
-      </plugin>
-    </gazebo>
-  </xacro:if>
-  <xacro:if value="$(arg front_laser)">
-    <husky_part parent="base_link_front_bumper_part" name="sick_bracket" mesh="lidar_mount"
-      colour="DarkGray"
-      translateX="-0.12" translateY="0" translateZ="0"
-      rotateX="0" rotateY="0.0" rotateZ="0"/>
-      <gazebo reference="lidar_mount_bracket_part">
-        <material>Gazebo/DarkGrey</material>
-      </gazebo>
-      <xacro:sick_lms100 prefix="front" />
-      <joint name="front_laser_joint" type="fixed">
-        <origin xyz="0.07 0 0.17" rpy="0 0 0" />
-        <parent link="base_link_front_bumper_part_sick_bracket_part" />
-        <child link="front_laser" />
-      </joint>
-    </xacro:if>
-  </robot>
+  <xacro:husky_wheel prefix="front_left">
+    <origin xyz="${wheelbase/2} ${track/2} ${wheel_vertical_offset}" rpy="0 0 0" />
+  </xacro:husky_wheel>
+  <xacro:husky_wheel prefix="front_right">
+    <origin xyz="${wheelbase/2} ${-track/2} ${wheel_vertical_offset}" rpy="0 0 0" />
+  </xacro:husky_wheel>
+  <xacro:husky_wheel prefix="rear_left">
+    <origin xyz="${-wheelbase/2} ${track/2} ${wheel_vertical_offset}" rpy="0 0 0" />
+  </xacro:husky_wheel>
+  <xacro:husky_wheel prefix="rear_right">
+    <origin xyz="${-wheelbase/2} ${-track/2} ${wheel_vertical_offset}" rpy="0 0 0" />
+  </xacro:husky_wheel>
+</robot>

File: urdf/parts.urdf.xacro (robot description, xacro)
@@ -32,45 +32,131 @@
 	xmlns:interface="http://playerstage.sourceforge.net/gazebo/xmlschema/#interface"
 	xmlns:xacro="http://ros.org/wiki/xacro" name="husky_part">
-	<property name="x_com" value="0.00000000" /> <!-- com : center of mass -->
-	<property name="y_com" value="0.00000000" /> <!-- com : center of mass -->
-	<property name="z_com" value="0.00000000" /> <!-- com : center of mass -->
-	<property name="x_size" value="1.0" />
-	<property name="y_size" value="1.0" />
-	<property name="z_size" value="1.0" />
-	<property name="mass" value="0.1" /> <!-- in kg-->
-	<property name="ixx_com_cs" value="0.01" /> <!-- at center of mass aligned with coordinate system, kg*m^2-->
-	<property name="ixy_com_cs" value="0.0" /> <!-- at center of mass aligned with coordinate system, kg*m^2-->
-	<property name="ixz_com_cs" value="0.0" /> <!-- at center of mass aligned with coordinate system, kg*m^2-->
-	<property name="iyy_com_cs" value="0.01" /> <!-- at center of mass aligned with coordinate system, kg*m^2-->
-	<property name="iyz_com_cs" value="0.00" /> <!-- at center of mass aligned with coordinate system, kg*m^2-->
-	<property name="izz_com_cs" value="0.01" /> <!-- at center of mass aligned with coordinate system, kg*m^2-->
-	<xacro:macro name="husky_part" params="parent name mesh colour translateX translateY translateZ rotateX rotateY rotateZ">
-		<link name="${parent}_${name}_part">
-			<inertial>
-				<mass value="${mass}" />
-				<origin xyz="${x_com} ${y_com} ${z_com}" />
-				<inertia ixx="${ixx_com_cs}" ixy="${ixy_com_cs}" ixz="${ixz_com_cs}"
-					iyy="${iyy_com_cs}" iyz="${iyz_com_cs}" izz="${izz_com_cs}" />
-			</inertial>
-			<visual>
-				<origin xyz="0 0 0" rpy="0 0 0" />
-				<geometry>
-					<mesh filename="package://husky_description/meshes/${mesh}.stl" />
-				</geometry>
-				<material name="${colour}" />
-			</visual>
-			<collision>
-				<origin xyz="0 0 0" rpy="0 0 0"/>
-				<geometry>
-					<box size="0.001 0.001 0.001" /> <!--the collision boundary for parts are taken into account by collision boundary of the base_link-->
-				</geometry>
-			</collision>
-		</link>
-		<joint name="${parent}_${name}_joint" type="fixed">
-		    <origin xyz="${translateX} ${translateY} ${translateZ}"
-		            rpy="${rotateX} ${rotateY} ${rotateZ}" />
-		    <parent link="${parent}" />
-		    <child link="${parent}_${name}_part" />
-		</joint>
-  	</xacro:macro>
+<!-- DECORATIONS -->
+  <!-- Top Plate -->
+  <link name="top_plate_link">
+    <visual>
+      <origin xyz="0 0 0" rpy="0 0 0" />
+      <geometry>
+        <mesh filename="package://husky_description/meshes/top_plate.stl" />
+      </geometry>
+      <material name="Yellow" />
+    </visual>
+  </link>
+  <joint name="top_plate" type="fixed">
+    <parent link="base_link" />
+    <child link="top_plate_link" />
+  </joint>
+  <gazebo reference="top_plate_link">
+    <material>Gazebo/Yellow</material>
+  </gazebo>
+  <link name="user_rail_link">
+    <visual>
+      <geometry>
+        <mesh filename="package://husky_description/meshes/user_rail.stl" />
+      </geometry>
+      <material name="DarkGray" />
+    </visual>
+  </link>
+  <joint name="user_rail" type="fixed">
+    <origin xyz="0.272 0 0.245" rpy="0 0 0" />
+    <parent link="base_link" />
+    <child link="user_rail_link" />
+  </joint>
+  <gazebo reference="user_rail_link">
+    <material>Gazebo/DarkGray</material>
+  </gazebo>
+  <link name="front_bumper_link">
+    <visual>
+      <geometry>
+        <mesh filename="package://husky_description/meshes/bumper.stl" />
+      </geometry>
+      <material name="DarkGray" />
+    </visual>
+  </link>
+  <joint name="front_bumper" type="fixed">
+    <origin xyz="0.48 0 0.091" rpy="0 0 0" />
+    <parent link="base_link" />
+    <child link="front_bumper_link" />
+  </joint>
+  <gazebo reference="front_bumper_link">
+    <material>Gazebo/DarkGray</material>
+  </gazebo>
+  <link name="rear_bumper_link">
+    <visual>
+      <geometry>
+        <mesh filename="package://husky_description/meshes/bumper.stl" />
+      </geometry>
+      <material name="DarkGray" />
+    </visual>
+  </link>
+  <joint name="rear_bumper" type="fixed">
+    <origin xyz="-0.48 0 0.091" rpy="0 0 ${M_PI}" />
+    <parent link="base_link" />
+    <child link="rear_bumper_link" />
+  </joint>
+  <gazebo reference="rear_bumper_link">
+    <material>Gazebo/DarkGray</material>
+  </gazebo>
+  <gazebo>
+    <plugin name="gazebo_ros_control" filename="libgazebo_ros_control.so">
+      <robotNamespace>/</robotNamespace>
+    </plugin>
+  </gazebo>
+  <xacro:if value="$(arg imu_enabled)">
+    <gazebo>
+      <plugin name="imu_controller" filename="libhector_gazebo_ros_imu.so">
+        <robotNamespace>/</robotNamespace>
+        <updateRate>50.0</updateRate>
+        <bodyName>base_link</bodyName>
+        <topicName>imu/data</topicName>
+        <accelDrift>0.005 0.005 0.005</accelDrift>
+        <accelGaussianNoise>0.005 0.005 0.005</accelGaussianNoise>
+        <rateDrift>0.005 0.005 0.005 </rateDrift>
+        <rateGaussianNoise>0.005 0.005 0.005 </rateGaussianNoise>
+        <headingDrift>0.005</headingDrift>
+        <headingGaussianNoise>0.005</headingGaussianNoise>
+      </plugin>
+    </gazebo>
+  </xacro:if>
+  <xacro:if value="$(arg gps_enabled)">
+    <gazebo>
+      <plugin name="gps_controller" filename="libhector_gazebo_ros_gps.so">
+        <updateRate>40</updateRate>
+        <robotNamespace>/</robotNamespace>
+        <bodyName>base_link</bodyName>
+        <frameId>base_link</frameId>
+        <topicName>/navsat/fix</topicName>
+        <velocityTopicName>/navsat/vel</velocityTopicName>
+        <referenceLatitude>49.9</referenceLatitude>
+        <referenceLongitude>8.9</referenceLongitude>
+        <referenceHeading>0</referenceHeading>
+        <referenceAltitude>0</referenceAltitude>
+        <drift>0.0001 0.0001 0.0001</drift>
+      </plugin>
+    </gazebo>
+  </xacro:if>
+  <xacro:if value="$(arg front_laser)">
+    <link name="sick_bracket_link">
+      <visual>
+        <geometry>
+          <mesh filename="package://husky_description/meshes/lidar_mount.stl" />
+        </geometry>
+        <material name="DarkGray" />
+      </visual>
+    </link>
+    <joint name="sick_bracket" type="fixed">
+      <origin xyz="-0.12 0 0" rpy="0 0 0" />
+      <parent link="front_bumper_link" />
+      <child link="sick_bracket_link" />
+    </joint>
+    <gazebo reference="sick_bracket_link">
+      <material>Gazebo/DarkGray</material>
+    </gazebo>
+    <xacro:sick_lms100 prefix="front" />
+    <joint name="front_laser_joint" type="fixed">
+      <origin xyz="0.07 0 0.17" rpy="0 0 0" />
+      <parent link="sick_bracket_link" />
+      <child link="front_laser" />
+    </joint>
+  </xacro:if>
 </robot>

File: urdf/wheel.urdf.xacro (robot description, xacro)
@@ -27,31 +27,13 @@
 <robot xmlns:xacro="http://ros.org/wiki/xacro" name="husky_wheel">
 	<property name="M_PI" value="3.14159"/>
-	<!-- Wheel -->
-	<property name="wheel_x_com" value="0.00000000" /> <!-- com : center of mass -->
-	<property name="wheel_y_com" value="0.00000000" /> <!-- com : center of mass -->
-	<property name="wheel_z_com" value="0.00019000" /> <!-- com : center of mass -->
-	<property name="wheel_x_size" value="0.35550000" />
-	<property name="wheel_y_size" value="0.35550000" />
-	<property name="wheel_z_size" value="0.11430000" />
-	<property name="wheel_mass" value="2.63657000" /> <!-- in kg-->
-	<property name="wheel_ixx_com_cs" value="0.02466885" /> <!-- at center of mass aligned with coordinate system, kg*m^2-->
-	<property name="wheel_ixy_com_cs" value="0.00000000" /> <!-- at center of mass aligned with coordinate system, kg*m^2-->
-	<property name="wheel_ixz_com_cs" value="0.00000000" /> <!-- at center of mass aligned with coordinate system, kg*m^2-->
-	<property name="wheel_iyy_com_cs" value="0.02466885" /> <!-- at center of mass aligned with coordinate system, kg*m^2-->
-	<property name="wheel_iyz_com_cs" value="0.00000000" /> <!-- at center of mass aligned with coordinate system, kg*m^2-->
-	<property name="wheel_izz_com_cs" value="0.04410576" /> <!-- at center of mass aligned with coordinate system, kg*m^2-->
-	<property name="base_x_origin_to_wheel_origin" value="0.25600006" />
-	<property name="base_y_origin_to_wheel_origin" value="0.285475" />
-	<property name="base_z_origin_to_wheel_origin" value="0.03282508" />
-	<xacro:macro name="husky_wheel" params="fb lr parent translateX translateY flipY"> <!--fb : front, back ; lr: left, right -->
-		<link name="${fb}_${lr}_wheel">
+	<xacro:macro name="husky_wheel" params="prefix *joint_pose">
+		<link name="${prefix}_wheel_link">
 			<inertial>
-				<mass value="${wheel_mass}" />
-				<origin xyz="${wheel_x_com} ${wheel_y_com} ${wheel_z_com}" />
-				<inertia  ixx="${wheel_ixx_com_cs}" ixy="${wheel_ixy_com_cs}" ixz="${wheel_ixz_com_cs}"
-					iyy="${wheel_iyy_com_cs}" iyz="${wheel_iyz_com_cs}" izz="${wheel_izz_com_cs}" />
+				<mass value="2.637" />
+				<origin xyz="0 0 0" />
+				<inertia  ixx="0.02467" ixy="0" ixz="0" iyy="0.02467" iyz="0" izz="0.04411" />
 			</inertial>
 			<visual>
-				<origin xyz="0 0 0" rpy="${flipY*M_PI} 0 0" />
+				<origin xyz="0 0 0" rpy="0 0 0" />
 				<geometry>
 					<mesh filename="package://husky_description/meshes/wheel.stl" />
@@ -60,36 +42,33 @@
 			</visual>
 			<collision>
-				<origin xyz="0 0 0" rpy="${flipY*M_PI/2} 0 0" />
+				<origin xyz="0 0 0" rpy="${M_PI/2} 0 0" />
 				<geometry>
-				    <cylinder length="${wheel_z_size}" radius="${wheel_x_size/2}" />
+				    <cylinder length="0.1143" radius="0.3555" />
 				</geometry>
 			</collision>
 		</link>
-		<gazebo reference="${fb}_${lr}_wheel">
+		<gazebo reference="${prefix}_wheel_link">
 			<mu1 value="1.0"/>
 			<mu2 value="1.0"/>
-			<kp  value="10000000.0" />
-			<kd  value="1.0" />
+			<kp value="10000000.0" />
+			<kd value="1.0" />
 			<fdir1 value="1 0 0"/>
 			<material>Gazebo/Grey</material>
 			<turnGravityOff>false</turnGravityOff>
 		</gazebo>
-		<joint name="joint_${fb}_${lr}_wheel" type="continuous">
-			<parent link="${parent}"/>
-			<child link="${fb}_${lr}_wheel"/>
-			<origin xyz="${translateX * base_x_origin_to_wheel_origin} ${translateY * base_y_origin_to_wheel_origin} ${base_z_origin_to_wheel_origin}" rpy="0 0 0" />
+		<joint name="${prefix}_wheel" type="continuous">
+			<parent link="base_link"/>
+			<child link="${prefix}_wheel_link"/>
+			<xacro:insert_block name="joint_pose"/>
 			<axis xyz="0 1 0" rpy="0 0 0" />
-			<limit effort="100" velocity="100"/>
-			<joint_properties damping="0.0" friction="0.0"/>
 		</joint>
-		<!-- Transmission is important to link the joints and the controller -->
-		<transmission name="joint_${fb}_${lr}_wheel_trans" type="SimpleTransmission">
+		<transmission name="${prefix}_wheel_trans" type="SimpleTransmission">
 			<type>transmission_interface/SimpleTransmission</type>
-			<joint name="joint_${fb}_${lr}_wheel">
+			<actuator name="${prefix}_wheel_motor">
+				<mechanicalReduction>1</mechanicalReduction>
+			</actuator>
+			<joint name="${prefix}_wheel">
 				<hardwareInterface>VelocityJointInterface</hardwareInterface>
 			</joint>
-			<actuator name="joint_${fb}_${lr}_wheel_actuator">
-				<mechanicalReduction>1</mechanicalReduction>
-			</actuator>
 		</transmission>
   	</xacro:macro>
