Commit message: RP-248 Add imu_link to urdf

File: urdf/base.urdf.xacro (robot description, xacro)
@@ -5,8 +5,5 @@
   <xacro:include filename="$(find husky_description)/urdf/wheel.urdf.xacro" />
   <xacro:include filename="$(find husky_description)/urdf/parts.urdf.xacro" />
-  <xacro:include filename="$(find husky_description)/urdf/sensors/gps.urdf.xacro" />
   <xacro:include filename="$(find husky_description)/urdf/sensors/sick_lms100.urdf.xacro" />
-  <!-- PROPERTY LIST -->
-  <property name="M_PI" value="3.1415926535897931" />
   <!-- Size of the base. -->
   <property name="base_x_size" value="0.98740000" />

File: urdf/parts.urdf.xacro (robot description, xacro)
@@ -32,70 +32,40 @@
 	xmlns:interface="http://playerstage.sourceforge.net/gazebo/xmlschema/#interface"
 	xmlns:xacro="http://ros.org/wiki/xacro" name="husky_part">
-<!-- DECORATIONS -->
-  <!-- Top Plate -->
-  <link name="top_plate_link">
-    <visual>
-      <origin xyz="0 0 0" rpy="0 0 0" />
-      <geometry>
-        <mesh filename="package://husky_description/meshes/top_plate.stl" />
-      </geometry>
-      <material name="Yellow" />
-    </visual>
-  </link>
-  <joint name="top_plate" type="fixed">
+  <!-- PROPERTY LIST -->
+  <property name="M_PI" value="3.1415926535897931" />
+  <link name="imu_link"/>
+  <joint name="imu_joint" type="fixed">
+    <origin xyz="0 0 0" rpy="${M_PI/2} ${M_PI/2} 0" />
     <parent link="base_link" />
-    <child link="top_plate_link" />
+    <child link="imu_link" />
   </joint>
-  <gazebo reference="top_plate_link">
-    <material>Gazebo/Yellow</material>
+  <gazebo reference="imu_link">
+    <turnGravityOff>false</turnGravityOff>
   </gazebo>
-  <link name="user_rail_link">
-    <visual>
-      <geometry>
-        <mesh filename="package://husky_description/meshes/user_rail.stl" />
-      </geometry>
-      <material name="DarkGrey" />
-    </visual>
-  </link>
-  <joint name="user_rail" type="fixed">
-    <origin xyz="0.272 0 0.245" rpy="0 0 0" />
-    <parent link="base_link" />
-    <child link="user_rail_link" />
-  </joint>
-  <gazebo reference="user_rail_link">
-    <material>Gazebo/DarkGrey</material>
-  </gazebo>
-  <link name="front_bumper_link">
-    <visual>
-      <geometry>
-        <mesh filename="package://husky_description/meshes/bumper.stl" />
-      </geometry>
-      <material name="DarkGrey" />
-    </visual>
-  </link>
-  <joint name="front_bumper" type="fixed">
-    <origin xyz="0.48 0 0.091" rpy="0 0 0" />
-    <parent link="base_link" />
-    <child link="front_bumper_link" />
-  </joint>
-  <gazebo reference="front_bumper_link">
-    <material>Gazebo/DarkGrey</material>
-  </gazebo>
-  <link name="rear_bumper_link">
-    <visual>
-      <geometry>
-        <mesh filename="package://husky_description/meshes/bumper.stl" />
-      </geometry>
-      <material name="DarkGrey" />
-    </visual>
-  </link>
-  <joint name="rear_bumper" type="fixed">
-    <origin xyz="-0.48 0 0.091" rpy="0 0 ${M_PI}" />
-    <parent link="base_link" />
-    <child link="rear_bumper_link" />
-  </joint>
-  <gazebo reference="rear_bumper_link">
-    <material>Gazebo/DarkGrey</material>
-  </gazebo>
+  <xacro:if value="$(arg front_laser)">
+    <link name="sick_bracket_link">
+      <visual>
+        <geometry>
+          <mesh filename="package://husky_description/meshes/lidar_mount.stl" />
+        </geometry>
+        <material name="DarkGrey" />
+      </visual>
+    </link>
+    <joint name="sick_bracket" type="fixed">
+      <origin xyz="-0.12 0 0" rpy="0 0 0" />
+      <parent link="front_bumper_link" />
+      <child link="sick_bracket_link" />
+    </joint>
+    <gazebo reference="sick_bracket_link">
+      <material>Gazebo/DarkGrey</material>
+      <turnGravityOff>false</turnGravityOff>
+    </gazebo>
+    <xacro:sick_lms100 prefix="front" />
+    <joint name="front_laser_joint" type="fixed">
+      <origin xyz="0.07 0 0.17" rpy="0 0 0" />
+      <parent link="sick_bracket_link" />
+      <child link="front_laser" />
+    </joint>
+  </xacro:if>
   <gazebo>
     <plugin name="gazebo_ros_control" filename="libgazebo_ros_control.so">
@@ -136,27 +106,72 @@
     </gazebo>
   </xacro:if>
-  <xacro:if value="$(arg front_laser)">
-    <link name="sick_bracket_link">
-      <visual>
-        <geometry>
-          <mesh filename="package://husky_description/meshes/lidar_mount.stl" />
-        </geometry>
-        <material name="DarkGrey" />
-      </visual>
-    </link>
-    <joint name="sick_bracket" type="fixed">
-      <origin xyz="-0.12 0 0" rpy="0 0 0" />
-      <parent link="front_bumper_link" />
-      <child link="sick_bracket_link" />
-    </joint>
-    <gazebo reference="sick_bracket_link">
-      <material>Gazebo/DarkGrey</material>
-    </gazebo>
-    <xacro:sick_lms100 prefix="front" />
-    <joint name="front_laser_joint" type="fixed">
-      <origin xyz="0.07 0 0.17" rpy="0 0 0" />
-      <parent link="sick_bracket_link" />
-      <child link="front_laser" />
-    </joint>
-  </xacro:if>
+<!-- DECORATIONS -->
+  <link name="top_plate_link">
+    <visual>
+      <origin xyz="0 0 0" rpy="0 0 0" />
+      <geometry>
+        <mesh filename="package://husky_description/meshes/top_plate.stl" />
+      </geometry>
+      <material name="Yellow" />
+    </visual>
+  </link>
+  <joint name="top_plate" type="fixed">
+    <parent link="base_link" />
+    <child link="top_plate_link" />
+  </joint>
+  <gazebo reference="top_plate_link">
+    <material>Gazebo/Yellow</material>
+    <turnGravityOff>false</turnGravityOff>
+  </gazebo>
+  <link name="user_rail_link">
+    <visual>
+      <geometry>
+        <mesh filename="package://husky_description/meshes/user_rail.stl" />
+      </geometry>
+      <material name="DarkGrey" />
+    </visual>
+  </link>
+  <joint name="user_rail" type="fixed">
+    <origin xyz="0.272 0 0.245" rpy="0 0 0" />
+    <parent link="base_link" />
+    <child link="user_rail_link" />
+  </joint>
+  <gazebo reference="user_rail_link">
+    <material>Gazebo/DarkGrey</material>
+    <turnGravityOff>false</turnGravityOff>
+  </gazebo>
+  <link name="front_bumper_link">
+    <visual>
+      <geometry>
+        <mesh filename="package://husky_description/meshes/bumper.stl" />
+      </geometry>
+      <material name="DarkGrey" />
+    </visual>
+  </link>
+  <joint name="front_bumper" type="fixed">
+    <origin xyz="0.48 0 0.091" rpy="0 0 0" />
+    <parent link="base_link" />
+    <child link="front_bumper_link" />
+  </joint>
+  <gazebo reference="front_bumper_link">
+    <material>Gazebo/DarkGrey</material>
+    <turnGravityOff>false</turnGravityOff>
+  </gazebo>
+  <link name="rear_bumper_link">
+    <visual>
+      <geometry>
+        <mesh filename="package://husky_description/meshes/bumper.stl" />
+      </geometry>
+      <material name="DarkGrey" />
+    </visual>
+  </link>
+  <joint name="rear_bumper" type="fixed">
+    <origin xyz="-0.48 0 0.091" rpy="0 0 ${M_PI}" />
+    <parent link="base_link" />
+    <child link="rear_bumper_link" />
+  </joint>
+  <gazebo reference="rear_bumper_link">
+    <material>Gazebo/DarkGrey</material>
+    <turnGravityOff>false</turnGravityOff>
+  </gazebo>
 </robot>

Commit message: RP-248 refactor links with chassis_link

File: urdf/base.urdf.xacro (robot description, xacro)
@@ -12,8 +12,14 @@
   <!-- Inertial values for the base at center of mass, aligned with coordinate system. Units are kg*m^2 -->
   <xacro:property name="wheelbase" value="0.5120" />
+  <xacro:property name="wheelbase" value="0.5120" />
   <xacro:property name="track" value="0.5708" />
   <xacro:property name="wheel_vertical_offset" value="0.03282" />
   <!-- Root node is the body of the robot. -->
-  <link name="base_link">
+  <link name="base_link"/>
+  <gazebo reference="base_link">
+    <material>Gazebo/DarkGrey</material>
+    <turnGravityOff>false</turnGravityOff>
+  </gazebo>
+  <link name="chassis_link">
     <visual>
       <origin xyz="0 0 0" rpy="0 0 0" />
@@ -30,10 +36,4 @@
       </geometry>
     </collision>
-  </link>
-  <gazebo reference="base_link">
-    <material>Gazebo/DarkGrey</material>
-    <turnGravityOff>false</turnGravityOff>
-  </gazebo>
-  <link name="base_inertia">
     <inertial>
       <mass value="33.455" />
@@ -43,10 +43,10 @@
      </inertial>
    </link>
-   <joint name="base_inertia_joint" type="fixed">
-    <origin xyz="0 0 0" rpy="0 0 0" />
+   <joint name="chassis_joint" type="fixed">
+    <origin xyz="0 0 ${0.17775 - wheel_vertical_offset}" rpy="0 0 0" />
     <parent link="base_link" />
-    <child link="base_inertia" />
+    <child link="chassis_link" />
   </joint>
-  <gazebo reference="base_inertia">
+  <gazebo reference="chassis_link">
     <turnGravityOff>false</turnGravityOff>
   </gazebo>

File: urdf/parts.urdf.xacro (robot description, xacro)
@@ -36,6 +36,6 @@
   <link name="imu_link"/>
   <joint name="imu_joint" type="fixed">
-    <origin xyz="0 0 0" rpy="${M_PI/2} ${M_PI/2} 0" />
-    <parent link="base_link" />
+    <origin xyz="$(optenv HUSKY_IMU_XYZ 0.25 0 0.0415)" rpy="$(optenv HUSKY_IMU_RPY 0 -1.57 0)" />
+    <parent link="chassis_link" />
     <child link="imu_link" />
   </joint>
@@ -117,5 +117,5 @@
   </link>
   <joint name="top_plate" type="fixed">
-    <parent link="base_link" />
+    <parent link="chassis_link" />
     <child link="top_plate_link" />
   </joint>
@@ -134,5 +134,5 @@
   <joint name="user_rail" type="fixed">
     <origin xyz="0.272 0 0.245" rpy="0 0 0" />
-    <parent link="base_link" />
+    <parent link="chassis_link" />
     <child link="user_rail_link" />
   </joint>
@@ -151,5 +151,5 @@
   <joint name="front_bumper" type="fixed">
     <origin xyz="0.48 0 0.091" rpy="0 0 0" />
-    <parent link="base_link" />
+    <parent link="chassis_link" />
     <child link="front_bumper_link" />
   </joint>
@@ -168,5 +168,5 @@
   <joint name="rear_bumper" type="fixed">
     <origin xyz="-0.48 0 0.091" rpy="0 0 ${M_PI}" />
-    <parent link="base_link" />
+    <parent link="chassis_link" />
     <child link="rear_bumper_link" />
   </joint>

File: urdf/wheel.urdf.xacro (robot description, xacro)
@@ -58,5 +58,5 @@
 		</gazebo>
 		<joint name="${prefix}_wheel" type="continuous">
-			<parent link="base_link"/>
+			<parent link="chassis_link"/>
 			<child link="${prefix}_wheel_link"/>
 			<xacro:insert_block name="joint_pose"/>

Commit message: RP-264 Fix up Husky URDF

File: urdf/base.urdf.xacro (robot description, xacro)
@@ -10,9 +10,9 @@
   <property name="base_y_size" value="0.57090000" />
   <property name="base_z_size" value="0.24750000" />
-  <!-- Inertial values for the base at center of mass, aligned with coordinate system. Units are kg*m^2 -->
-  <xacro:property name="wheelbase" value="0.5120" />
   <xacro:property name="wheelbase" value="0.5120" />
   <xacro:property name="track" value="0.5708" />
   <xacro:property name="wheel_vertical_offset" value="0.03282" />
+  <xacro:property name="wheel_length" value="0.1143" />
+  <xacro:property name="wheel_radius" value="0.17775" />
   <!-- Root node is the body of the robot. -->
   <link name="base_link"/>
@@ -44,5 +44,5 @@
    </link>
    <joint name="chassis_joint" type="fixed">
-    <origin xyz="0 0 ${0.17775 - wheel_vertical_offset}" rpy="0 0 0" />
+    <origin xyz="0 0 ${wheel_radius - wheel_vertical_offset}" rpy="0 0 0" />
     <parent link="base_link" />
     <child link="chassis_link" />

File: urdf/parts.urdf.xacro (robot description, xacro)
@@ -36,5 +36,5 @@
   <link name="imu_link"/>
   <joint name="imu_joint" type="fixed">
-    <origin xyz="$(optenv HUSKY_IMU_XYZ 0.25 0 0.0415)" rpy="$(optenv HUSKY_IMU_RPY 0 1.5708 1.5708)" />
+    <origin xyz="$(optenv HUSKY_IMU_XYZ 0.25 0 0.0415)" rpy="$(optenv HUSKY_IMU_RPY 1.5708 0 -1.5708)" />
     <parent link="chassis_link" />
     <child link="imu_link" />

File: urdf/wheel.urdf.xacro (robot description, xacro)
@@ -44,5 +44,5 @@
 				<origin xyz="0 0 0" rpy="${M_PI/2} 0 0" />
 				<geometry>
-				    <cylinder length="0.1143" radius="0.17775" />
+				    <cylinder length="${wheel_length}" radius="${wheel_radius}" />
 				</geometry>
 			</collision>
